Commit message: casi queda falta que compile

File: xarm_description/urdf/xarm.urdf (robot description, URDF)
Before this commit: robot xArm, 2 links, 1 joints
Links:
- removed link xArm_5_link
- removed link xArm_6_link
- added link xarm_2_link; collision mesh filename=package://xarm_description/meshes/stls/link2.stl scale=1.0 1.0 1.0; visual mesh filename=package://xarm_description/meshes/stls/link2.stl scale=1.0 1.0 1.0
- added link xarm_3_link; collision mesh filename=package://xarm_description/meshes/stls/link3.stl scale=1.0 1.0 1.0; visual mesh filename=package://xarm_description/meshes/stls/link3.stl scale=1.0 1.0 1.0
- added link xarm_4_link; collision mesh filename=package://xarm_description/meshes/stls/link4.stl scale=1.0 1.0 1.0; visual mesh filename=package://xarm_description/meshes/stls/link4.stl scale=1.0 1.0 1.0
- added link xarm_5_link; collision mesh filename=package://xarm_description/meshes/stls/link5.stl scale=1.0 1.0 1.0; visual mesh filename=package://xarm_description/meshes/stls/link5.stl scale=1.0 1.0 1.0
- added link xarm_6_link; collision mesh filename=package://xarm_description/meshes/stls/link6.stl scale=1.0 1.0 1.0; visual mesh filename=package://xarm_description/meshes/stls/link6.stl scale=1.0 1.0 1.0
- added link xarm_base_link; collision mesh filename=package://xarm_description/meshes/stls/base.stl scale=1.0 1.0 1.0; visual mesh filename=package://xarm_description/meshes/stls/base.stl scale=1.0 1.0 1.0
Joints:
- removed joint xArm_6_joint
- added joint xarm_2_joint: type revolute, parent xarm_3_link, child xarm_2_link, origin xyz=0 -0.001205 0.05306 rpy=0 0 0, axis 1 0 0, limit lower=-1.5 upper=1.5 effort=1000 velocity=0.5
- added joint xarm_3_joint: type revolute, parent xarm_4_link, child xarm_3_link, origin xyz=0 0.0 0.09825 rpy=0 0 0, axis 1 0 0, limit lower=-1.5 upper=1.5 effort=1000 velocity=0.5
- added joint xarm_4_joint: type revolute, parent xarm_5_link, child xarm_4_link, origin xyz=0 0.0 0.09765 rpy=0 0 0, axis 1 0 0, limit lower=-1.5 upper=1.5 effort=1000 velocity=0.5
- added joint xarm_5_joint: type revolute, parent xarm_6_link, child xarm_5_link, origin xyz=0 -0.0022 0.03195 rpy=0 0 0, axis 1 0 0, limit lower=-1.5 upper=1.5 effort=1000 velocity=0.5
- added joint xarm_6_joint: type revolute, parent xarm_base_link, child xarm_6_link, origin xyz=0 0.0 0.03603 rpy=0 0 0, axis 1 0 0, limit lower=-1.5 upper=1.5 effort=1000 velocity=0.5

Commit message: Moveit controller ready

File: xarm_description/urdf/xarm.urdf (robot description, URDF)
Before this commit: robot xarm, 6 links, 5 joints
Links:
- link xarm_2_link: mass None -> 0.1
- link xarm_3_link: mass None -> 0.1
- link xarm_4_link: mass None -> 0.1
- link xarm_5_link: mass None -> 0.1
- link xarm_6_link: mass None -> 0.1
- link xarm_base_link: mass None -> 0.1
Joints:
- joint xarm_2_joint: axis 1 0 0 -> 0 0 1
- joint xarm_6_joint: axis 1 0 0 -> 0 0 1

Commit message: latest changes

File: xarm_description/urdf/xarm.urdf (robot description, URDF)
Before this commit: robot xarm, 6 links, 5 joints
Joints:
- joint xarm_2_joint: limit lower=-1.5 upper=1.5 effort=1000 velocity=0.5 -> lower=-2.17494876 upper=1.63121157 effort=1000 velocity=1.0
- joint xarm_3_joint: limit lower=-1.5 upper=1.5 effort=1000 velocity=0.5 -> lower=-1.740612146 upper=1.86797401 effort=1000 velocity=1.0
- joint xarm_4_joint: limit lower=-1.5 upper=1.5 effort=1000 velocity=0.5 -> lower=-1.910427965 upper=1.910427965 effort=1000 velocity=1.0
- joint xarm_5_joint: limit lower=-1.5 upper=1.5 effort=1000 velocity=0.5 -> lower=-1.592023304 upper=1.86797401 effort=1000 velocity=1.0
- joint xarm_6_joint: limit lower=-1.5 upper=1.5 effort=1000 velocity=0.5 -> lower=-1.737238322 upper=1.79965407 effort=1000 velocity=1.0
